File: eeg.kicad_pcb (KiCad board)
At the start: 2 copper layers, 81.4 x 54.9 mm, 225 parts, among them J1 Conn_01x05_Male, J10 USB_B_Mini, J2 Conn_01x05_Male, J3 Conn_01x05_Male, J4 Conn_01x05_Male, J5 Conn_01x10, J6 Conn_01x10_Male, J7 Conn_01x10_Male, SW3 EVQ-Q2K03W, U1 STM32F446RE, U12 RN4678-V_RM100, U2 ADS1299-8CHANNEL, U3 LD39050PU33R, U4 TPS60403DBVT, U5 TPS73225DBVT, U6 TPS72325DBVT, Y1 16.00Mhz

Commit message: Hardware Revision V2.0: fix STM32 supply short, ADS1299 SRB2/BIAS, RN4678 wakeup/keepout, and BOM updates
Parts:
- C1: value 10uF -> 1nF
- C42: value 2.2uF -> 4.7uF; footprint Capacitor_Tantalum_SMD:CP_EIA-1608-08_AVX-J_Pad1.25x1.05mm_HandSolder -> Capacitor_SMD:C_0603_1608Metric
- R20, R21, R22: value R_Small -> 270
Connections:
- U1 pad 12: +3V3 -> GNDA
- U1 pad 63: +3V3 -> GNDA
- U12 pad 5: Net-(U12-Pad5) -> +3V3
- U12 pad 9: Net-(U12-Pad9) -> Net-(R31-Pad2)
- U2 pad 18: Net-(U2-Pad18) -> /SRB2
- Y1 pad 2: Net-(C81-Pad1) -> GNDA
- Y1 pad 3: (no net) -> Net-(C81-Pad1)
- Y1 pad 4: (no net) -> GNDA
Routing:
- net /SRB2: track 2.46 -> 29.2 mm
- net Net-(R31-Pad2): track 31.5 -> 34.7 mm
- net +3V3: track 262.0 -> 264.4 mm
- net GNDA: track 196.7 -> 195.1 mm
- net Net-(C81-Pad1): track 12.8 -> 14.3 mm
