File: eeg.sch (KiCad schematic (older format))
At the start: 136 parts, among them J1 Conn_01x05_Male, J10 USB_B_Mini, J2 Conn_01x05_Male, J3 Conn_01x05_Male, J4 Conn_01x05_Male, J5 Conn_01x10, J6 Conn_01x10_Male, J7 Conn_01x10_Male, SW2 SW_DIP_x03, SW3 EVQ-Q2K03W, U1 STM32F446RE, U12 RN4678-V_RM100, U2 ADS1299-8, U3 LD39050PU33R, U4 TPS60403DBVT, U5 TPS73225DBVT, U6 TPS72325DBVT, Y1 16.00Mhz

Commit message: Hardware Revision V2.0: fix STM32 supply short, ADS1299 SRB2/BIAS, RN4678 wakeup/keepout, and BOM updates
Parts:
- C1: value 10uF -> 1nF
- C42: value 2.2uF -> 4.7uF; footprint Capacitor_Tantalum_SMD:CP_EIA-1608-08_AVX-J_Pad1.25x1.05mm_HandSolder -> Capacitor_SMD:C_0603_1608Metric
- C62: footprint Capacitor_SMD:C_0603_1608Metric -> TCA1C106M8R:RESC3216X65N
- C80, C81: footprint Capacitor_SMD:C_1206_3216Metric -> Capacitor_SMD:C_0603_1608Metric
- R31: footprint LED_SMD:LED_0805_2012Metric -> Resistor_SMD:R_0805_2012Metric
Connections:
- wire segments 443 -> 447
- no-connect marks 57 -> 54
Changed lines of the file:
@@
 F 0 "C80" V 11806 7760 20  0000 C CNN
 F 1 "9pF" V 11737 7700 20  0000 C CNN
-F 2 "Capacitor_SMD:C_1206_3216Metric" H 11850 7700 50  0001 C CNN
+F 2 "Capacitor_SMD:C_0603_1608Metric" H 11850 7700 50  0001 C CNN
 F 3 "~" H 11850 7700 50  0001 C CNN
 	1    11850 7700
@@
 F 0 "C81" V 11700 7400 20  0000 C CNN
 F 1 "9pF" V 11737 7400 20  0000 C CNN
-F 2 "Capacitor_SMD:C_1206_3216Metric" H 11850 7400 50  0001 C CNN
+F 2 "Capacitor_SMD:C_0603_1608Metric" H 11850 7400 50  0001 C CNN
 F 3 "~" H 11850 7400 50  0001 C CNN
 	1    11850 7400
@@
 P 1350 4800
 F 0 "C1" H 1442 4846 50  0000 L CNN
-F 1 "10uF" H 1442 4800 50  0000 L CNN
+F 1 "1nF" H 1442 4800 50  0000 L CNN
 F 2 "Capacitor_SMD:C_0603_1608Metric" H 1350 4800 50  0001 C CNN
 F 3 "~" H 1350 4800 50  0001 C CNN
@@
 Text Label 5450 9000 1    12   ~ 0
 SRB1
+Text Label 5550 9000 1    12   ~ 0
+SRB2
 Text Label 5550 6450 1    12   ~ 0
 BIASOUT
@@
 F 0 "C62" V 5782 9304 12  0000 C CNN
 F 1 "100uF" V 5718 9304 12  0000 C CNN
-F 2 "Capacitor_SMD:C_0603_1608Metric" H 5750 9250 50  0001 C CNN
+F 2 "TCA1C106M8R:RESC3216X65N" H 5750 9250 50  0001 C CNN
 F 3 "~" H 5750 9250 50  0001 C CNN
 	1    5750 9250
@@
 $EndComp
 Wire Wire Line
-	13200 5950 12550 5950
+	13200 6150 12550 6150
 Connection ~ 12350 5950
-Connection ~ 12550 5950
 Wire Wire Line
 	12550 5950 12350 5950
@@
 NoConn ~ 6450 8750
 NoConn ~ 6650 8750
-NoConn ~ 5550 9000
 NoConn ~ 5450 6450
 NoConn ~ 13050 1150
@@
 	12150 8300 11900 8300
 Connection ~ 12150 8300
-Connection ~ 12500 8300
 Wire Wire Line
 	12500 8300 12350 8300
@@
 	13100 6800 13100 6700
 Wire Wire Line
-	13200 5950 13200 6800
+	13200 6150 13200 6800
+Connection ~ 12550 6150
 Wire Wire Line
 	13300 6800 13300 6700
@@
 P 14400 9200
 F 0 "C42" H 14450 9250 12  0000 L CNN
-F 1 "2.2uF" H 14500 9200 12  0000 R CNN
-F 2 "Capacitor_Tantalum_SMD:CP_EIA-1608-08_AVX-J_Pad1.25x1.05mm_HandSolder" H 14400 9200 50  0001 C CNN
+F 1 "4.7uF" H 14500 9200 12  0000 R CNN
+F 2 "Capacitor_SMD:C_0603_1608Metric" H 14400 9200 50  0001 C CNN
 F 3 "~" H 14400 9200 50  0001 C CNN
 	1    14400 9200
@@
 	12500 8400 12700 8400
 Wire Wire Line
-	12700 8300 12500 8300
+	12700 8300 12600 8300
+Wire Wire Line
+	12600 8300 12600 8500
+Wire Wire Line
+	12600 8500 12350 8500
+Connection ~ 12350 8500
 NoConn ~ 12700 8200
 NoConn ~ 12700 8100
@@
 F 0 "R31" V 3650 7600 50  0000 C CNN
 F 1 "270" V 3550 7600 50  0000 C CNN
-F 2 "LED_SMD:LED_0805_2012Metric" H 3750 7600 50  0001 C CNN
+F 2 "Resistor_SMD:R_0805_2012Metric" H 3750 7600 50  0001 C CNN
 F 3 "~" H 3750 7600 50  0001 C CNN
 	1    3750 7600
@@
 Connection ~ 6750 6250
 NoConn ~ 1550 6800
-NoConn ~ 1550 6900
-NoConn ~ 1550 7000
+Wire Wire Line
+	1550 6900 1400 6900
+Wire Wire Line
+	1550 7000 1400 7000
+Text Label 1400 7000 2    20   ~ 0
+INT3V3
+$Comp
+L power:+3.3V #PWR0186
+U 1 1 611D1001
+P 1400 6900
+F 0 "#PWR0186" H 1400 6750 50  0001 C CNN
+F 1 "+3.3V" H 1400 7050 20  0000 C CNN
+F 2 "" H 1400 6900 50  0001 C CNN
+F 3 "" H 1400 6900 50  0001 C CNN
+	1    1400 6900
+	1    0    0    -1
+$EndComp
 Text GLabel 1400 7700 0    50   Input ~ 0
 P2.0
